Commit message: debuging

File: source/isaaclab_assets/data/robot/icarus/unimanual/urdf/icarus.urdf (robot description, URDF)
Before this commit: robot icarus_orca, 61 links, 60 joints
Links:
- link baringattacher_link8_1: geometry collision mesh filename=file:///home/orbit/ros2_ws/src/icarus_urdf_v2_copy_descript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 scale=0.001 0.001 0.001; visual mesh filename=file:///home/orbit/ros2_ws/src/icarus_urdf_v2_copy_descript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 scale=0.001 0.001 0.001
- link base_link: geometry collision mesh filename=file:///home/orbit/ros2_ws/src/icarus_urdf_v2_copy_descript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 scale=0.001 0.001 0.001; visual mesh filename=file:///home/orbit/ros2_ws/src/icarus_urdf_v2_copy_descript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 scale=0.001 0.001 0.001
- link bearinginner_link9_1: geometry collision mesh filename=file:///home/orbit/ros2_ws/src/icarus_urdf_v2_copy_descript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 scale=0.001 0.001 0.001; visual mesh filename=file:///home/orbit/ros2_ws/src/icarus_urdf_v2_copy_descript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 scale=0.001 0.001 0.001
- link bearingleft_link16_1: geometry collision mesh filename=file:///home/orbit/ros2_ws/src/icarus_urdf_v2_copy_descript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 scale=0.001 0.001 0.001; visual mesh filename=file:///home/orbit/ros2_ws/src/icarus_urdf_v2_copy_descript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 scale=0.001 0.001 0.001
- link bearingouter_link10_1: geometry collision mesh filename=file:///home/orbit/ros2_ws/src/icarus_urdf_v2_copy_descript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 scale=0.001 0.001 0.001; visual mesh filename=file:///home/orbit/ros2_ws/src/icarus_urdf_v2_copy_descript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 scale=0.001 0.001 0.001
- link bearingright_link14_1: geometry collision mesh filename=file:///home/orbit/ros2_ws/src/icarus_urdf_v2_copy_descript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 scale=0.001 0.001 0.001; visual mesh filename=file:///home/orbit/ros2_ws/src/icarus_urdf_v2_copy_descript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 scale=0.001 0.001 0.001
- link case_link5_1: geometry collision mesh filename=file:///home/orbit/ros2_ws/src/icarus_urdf_v2_copy_descript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 scale=0.001 0.001 0.001; visual mesh filename=file:///home/orbit/ros2_ws/src/icarus_urdf_v2_copy_descript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 scale=0.001 0.001 0.001
- link connector_link2_1: geometry collision mesh filename=file:///home/orbit/ros2_ws/src/icarus_urdf_v2_copy_descript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 scale=0.001 0.001 0.001; visual mesh filename=file:///home/orbit/ros2_ws/src/icarus_urdf_v2_copy_descript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 scale=0.001 0.001 0.001
- link elbowconnector_link15_1: geometry collision mesh filename=file:///home/orbit/ros2_ws/src/icarus_urdf_v2_copy_descript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 scale=0.001 0.001 0.001; visual mesh filename=file:///home/orbit/ros2_ws/src/icarus_urdf_v2_copy_descript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 scale=0.001 0.001 0.001
- link frame1_link11_1: geometry collision mesh filename=file:///home/orbit/ros2_ws/src/icarus_urdf_v2_copy_descript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 scale=0.001 0.001 0.001; visual mesh filename=file:///home/orbit/ros2_ws/src/icarus_urdf_v2_copy_descript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 scale=0.001 0.001 0.001
- link frame2_link12_1: geometry collision mesh filename=file:///home/orbit/ros2_ws/src/icarus_urdf_v2_copy_descript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 scale=0.001 0.001 0.001; visual mesh filename=file:///home/orbit/ros2_ws/src/icarus_urdf_v2_copy_descript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 scale=0.001 0.001 0.001
- link handconnector_link21_1: geometry collision mesh filename=file:///home/orbit/ros2_ws/src/icarus_urdf_v2_copy_descript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 scale=0.001 0.001 0.001; visual mesh filename=file:///home/orbit/ros2_ws/src/icarus_urdf_v2_copy_descript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 scale=0.001 0.001 0.001
- link innerbearing_link20_1: geometry collision mesh filename=file:///home/orbit/ros2_ws/src/icarus_urdf_v2_copy_descript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 scale=0.001 0.001 0.001; visual mesh filename=file:///home/orbit/ros2_ws/src/icarus_urdf_v2_copy_descript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 scale=0.001 0.001 0.001
- link motor2_link3_1: geometry collision mesh filename=file:///home/orbit/ros2_ws/src/icarus_urdf_v2_copy_descript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 scale=0.001 0.001 0.001; visual mesh filename=file:///home/orbit/ros2_ws/src/icarus_urdf_v2_copy_descript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 scale=0.001 0.001 0.001
- link motor3_link6_1: geometry collision mesh filename=file:///home/orbit/ros2_ws/src/icarus_urdf_v2_copy_descript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 scale=0.001 0.001 0.001; visual mesh filename=file:///home/orbit/ros2_ws/src/icarus_urdf_v2_copy_descript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 scale=0.001 0.001 0.001
- link motor4_link13_1: geometry collision mesh filename=file:///home/orbit/ros2_ws/src/icarus_urdf_v2_copy_descript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 scale=0.001 0.001 0.001; visual mesh filename=file:///home/orbit/ros2_ws/src/icarus_urdf_v2_copy_descript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 scale=0.001 0.001 0.001
- link motor5_link17_1: geometry collision mesh filename=file:///home/orbit/ros2_ws/src/icarus_urdf_v2_copy_descript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 scale=0.001 0.001 0.001; visual mesh filename=file:///home/orbit/ros2_ws/src/icarus_urdf_v2_copy_descript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 scale=0.001 0.001 0.001
- link outerbearing_link18_1: geometry collision mesh filename=file:///home/orbit/ros2_ws/src/icarus_urdf_v2_copy_descript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 scale=0.001 0.001 0.001; visual mesh filename=file:///home/orbit/ros2_ws/src/icarus_urdf_v2_copy_descript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 scale=0.001 0.001 0.001
- link slot_link7_1: geometry collision mesh filename=file:///home/orbit/ros2_ws/src/icarus_urdf_v2_copy_descript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 scale=0.001 0.001 0.001; visual mesh filename=file:///home/orbit/ros2_ws/src/icarus_urdf_v2_copy_descript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 scale=0.001 0.001 0.001
- link uaconnector_link4_1: geometry collision mesh filename=file:///home/orbit/ros2_ws/src/icarus_urdf_v2_copy_descript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 scale=0.001 0.001 0.001; visual mesh filename=file:///home/orbit/ros2_ws/src/icarus_urdf_v2_copy_descript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 scale=0.001 0.001 0.001
